Commit message: Oculus Integration, Grabbing Objects, Hand Models

File: tutorials/pick_and_place/PickAndPlaceProject/Assets/URDF/niryo_one/niryo_one (1).urdf (robot description, URDF)
Before this commit: robot niryo_one (1), 15 links, 13 joints
Links:
- link arm_link: geometry collision mesh filename=package://meshes/arm_link.stl scale=5 5 5; visual mesh filename=package://meshes/arm_link.dae scale=5 5 5
- link base_link: geometry collision mesh filename=package://meshes/base_link.stl scale=5 5 5; visual mesh filename=package://meshes/base_link.dae scale=5 5 5
- link elbow_link: geometry collision mesh filename=package://meshes/elbow_link.stl scale=5 5 5; visual mesh filename=package://meshes/elbow_link.dae scale=5 5 5
- link forearm_link: geometry collision mesh filename=package://meshes/forearm_link.stl scale=5 5 5; visual mesh filename=package://meshes/forearm_link.dae scale=5 5 5
- link hand_link: geometry collision mesh filename=package://meshes/hand_link.stl scale=5 5 5; visual mesh filename=package://meshes/hand_link.dae scale=5 5 5
- link shoulder_link: geometry collision mesh filename=package://meshes/shoulder_link.stl scale=5 5 5; visual mesh filename=package://meshes/shoulder_link.dae scale=5 5 5
- link wrist_link: geometry collision mesh filename=package://meshes/wrist_link.stl scale=5 5 5; visual mesh filename=package://meshes/wrist_link.dae scale=5 5 5
